File: hardware/devboard/devboard.kicad_sch (KiCad schematic)
At the start: 20 parts, among them J10 ADC4, J11 ADC5, J12 ADC6, J13 ADC7, J2 TSW-126-07-L-D, J3 TSW-126-07-L-D, J5 I2C, J6 ADC0, J7 ADC1, J8 ADC2, J9 ADC3, SW1 434133025816, U3 W25Q128JVSIQ, U4 ILI9486_35_Shield

Commit message: feat(sch): add first schematic draft
Parts:
- removed C2: 100n, Capacitor_SMD:C_0603_1608Metric, symbol RPI_DB:Capacitors | MLCC | M1005/RP-01BJ9Y-KRGF41
- removed J2, J3: TSW-126-07-L-D, RPI_COMPILED:samtec_tsw-126-07-l-d, symbol RPI_DB:Connectors | Pin_Headers/RP-01KJ62-FD8Y6K
- removed MH1, MH2, MH3, MH4: NPTH FD2.75mm SM3.15mm KO6mm, RPI_COMPILED:none_mh_npth_fd2p75mm_sm3p15mm_ko6mm, symbol RPI_DB:Mechanical | Mounting_Holes/RP-01HF5R-LCTEJS
- removed R6: 1k, Resistor_SMD:R_0603_1608Metric, symbol RPI_DB:Resistors | Chip | M1005/RP-019A1P-4Z6ZWY
- removed SW1: 434133025816, RPI_COMPILED:wurthelek_434133025816, symbol RPI_DB:Electromechanical | Switches | Tactile/RP-01H0MT-6E9H8F
- removed U3: W25Q128JVSIQ, RPI_COMPILED:generic_soic127p790x195-8, symbol RPI_DB:Integrated_Circuits | Memory | Serial_Flash | SPI/RP-01JWD4-F1H4N9
- added C1, C5: 10u, Capacitor_SMD:C_0603_1608Metric, symbol RPI_DB:Capacitors | MLCC | M2012/RP-01GYSK-AVBE41
- added J14: Conn_01x02, Connector_PinSocket_2.54mm:PinSocket_1x02_P2.54mm_Vertical, symbol Connector_Generic:Conn_01x02
- added J4: Conn_01x03, Connector_PinSocket_2.54mm:PinSocket_1x03_P2.54mm_Vertical, symbol Connector_Generic:Conn_01x03
- added JP1: Jumper_3_Bridged12, Connector_PinSocket_2.54mm:PinSocket_1x03_P2.54mm_Vertical, symbol Jumper:Jumper_3_Bridged12
- added R1, R2, R3: 10k, Resistor_SMD:R_0805_2012Metric, symbol Device:R
- added SW1: RotaryEncoder_Switch_MP, Rotary_Encoder:RotaryEncoder_Alps_EC11E-Switch_Vertical_H20mm, symbol Device:RotaryEncoder_Switch_MP
- added U1: Core2350B0, Project Library:Core2350B0, symbol Project_Library:Core2350B0
- added U2: AMS1117CD-3.3, Package_TO_SOT_SMD:SOT-223-3_TabPin2, symbol Regulator_Linear:AMS1117CD-3.3
- added U5: (no value), Connector_PinHeader_2.54mm:PinHeader_1x03_P2.54mm_Vertical, symbol Project_Library:Boost_5V
- U4: footprint ILI9486_35_Shield:ILI9486_35_Shield -> Project Library:ILI9486_35_Shield
Connections:
- net +3V3: now also C5.1, R1.1, R2.1, R3.1, U1.3V3, U2.2 (VO)
- net GND: now also C1.2, C5.2, J14.2 (Pin_2), J4.2 (Pin_2), SW1.C, SW1.MP, SW1.S2, U1.GND, U2.1 (GND), U5.2 (GND)
- net GPIO0: now also U1.0 (GP0)
- net GPIO1: now also U1.1 (GP1)
- net GPIO10: now also U1.10 (GP10)
- net GPIO11: now also U1.11 (GP11)
- net GPIO12: now also U1.12 (GP12)
- net GPIO13: now also U1.13 (GP13)
- net GPIO14: now also U1.14 (GP14)
- net GPIO15: now also U1.15 (GP15)
- net GPIO16: now also U1.16 (GP16)
- net GPIO17: now also U1.17 (GP17)
- net GPIO18: now also U1.18 (GP18)
- net GPIO19: now also U1.19 (GP19)
- net GPIO2: now also U1.2 (GP2)
- net GPIO20: now also U1.20 (GP20)
- net GPIO21: now also U1.21 (GP21)
- net GPIO22: now also U1.22 (GP22)
- net GPIO23: now also U1.23 (GP23)
- net GPIO24: now also U1.24 (GP24)
- net GPIO25: now also U1.25 (GP25)
- net GPIO26: now also U1.26 (GP26)
- net GPIO27: now also R1.2, SW1.A, U1.27 (GP27)
- net GPIO28: now also U1.28 (GP28)
- net GPIO29: now also R2.2, SW1.B, U1.29 (GP29)
- net GPIO3: now also U1.3 (GP3)
- net GPIO30: now also R3.2, SW1.S1, U1.30 (GP30)
- net GPIO31: now also U1.31 (GP31)
- net GPIO32: now also U1.32 (GP32)
- net GPIO33: now also U1.33 (GP33)
- net GPIO34: now also U1.34 (GP34)
- net GPIO35: now also U1.35 (GP35)
- net GPIO36: now also U1.36 (GP36)
- net GPIO37: now also U1.37 (GP37)
- net GPIO38: now also U1.38 (GP38)
- net GPIO39: now also U1.39 (GP39)
- net GPIO4: now also U1.4 (GP4)
- net GPIO40_ADC0: now also U1.40 (GP40)
- net GPIO41_ADC1: now also U1.41 (GP41)
- net GPIO42_ADC2: now also U1.42 (GP42)
- net GPIO43_ADC3: now also U1.43 (GP43)
- net GPIO44_ADC4: now also U1.44 (GP44)
- net GPIO45_ADC5: now also U1.45 (GP45)
- net GPIO46_ADC6: now also U1.46 (GP46)
- net GPIO47_ADC7: now also U1.47 (GP47)
- net GPIO5: now also U1.5 (GP5)
- net GPIO6: now also U1.6 (GP6)
- net GPIO7: now also U1.7 (GP7)
- net GPIO8: now also U1.8 (GP8)
- net GPIO9: now also U1.9 (GP9)
- net SWCLK: now also J4.1 (Pin_1), U1.SWCLK
- net SWD: now also J4.3 (Pin_3), U1.SWDIO
- net VBUS: now also JP1.3 (B), U1.VBUS; no longer U4.19 (5V)
- new net +5V: JP1.1 (A), U5.3 (Vo)
- new net VBAT: J14.1 (Pin_1), U5.1 (Vi)
- new net VSYS: C1.1, JP1.2 (C), U2.3 (VI), U4.19 (5V)
- no-connect marks 1 -> 7
Other:
- removed sheet Power
- removed sheet RP2350B
- note added: "JST Debug Connector"
- note added: "Power"
- note removed: "BOOTSEL Button"
- note removed: "IOs"
- note removed: "Primary Flash"
- moved on the sheet: U4
